Commit message: changed to valid velocity limit

File: trunk/rtmros_common/hrpsys_gazebo/models/sandia_hand_right.urdf (robot description, URDF)
Before this commit: robot sandia_hand_right, 34 links, 33 joints
Joints:
- joint right_f0_j0: limit lower=-1.57079632679 upper=1.57079632679 effort=11 velocity=-1 -> lower=-1.57079632679 upper=1.57079632679 effort=11 velocity=24
- joint right_f0_j1: limit lower=-1.57079632679 upper=1.57079632679 effort=28 velocity=-1 -> lower=-1.57079632679 upper=1.57079632679 effort=28 velocity=24
- joint right_f0_j2: limit lower=-1.57079632679 upper=1.57079632679 effort=28 velocity=-1 -> lower=-1.57079632679 upper=1.57079632679 effort=28 velocity=24
- joint right_f1_j0: limit lower=-1.57079632679 upper=1.57079632679 effort=11 velocity=-1 -> lower=-1.57079632679 upper=1.57079632679 effort=11 velocity=24
- joint right_f1_j1: limit lower=-1.57079632679 upper=1.57079632679 effort=28 velocity=-1 -> lower=-1.57079632679 upper=1.57079632679 effort=28 velocity=24
- joint right_f1_j2: limit lower=-1.57079632679 upper=1.57079632679 effort=28 velocity=-1 -> lower=-1.57079632679 upper=1.57079632679 effort=28 velocity=24
- joint right_f2_j0: limit lower=-1.57079632679 upper=1.57079632679 effort=11 velocity=-1 -> lower=-1.57079632679 upper=1.57079632679 effort=11 velocity=24
- joint right_f2_j1: limit lower=-1.57079632679 upper=1.57079632679 effort=28 velocity=-1 -> lower=-1.57079632679 upper=1.57079632679 effort=28 velocity=24
- joint right_f2_j2: limit lower=-1.57079632679 upper=1.57079632679 effort=28 velocity=-1 -> lower=-1.57079632679 upper=1.57079632679 effort=28 velocity=24
- joint right_f3_j0: limit lower=-1.57079632679 upper=1.57079632679 effort=11 velocity=-1 -> lower=-1.57079632679 upper=1.57079632679 effort=11 velocity=24
- joint right_f3_j1: limit lower=-1.57079632679 upper=1.57079632679 effort=28 velocity=-1 -> lower=-1.57079632679 upper=1.57079632679 effort=28 velocity=24
- joint right_f3_j2: limit lower=-1.57079632679 upper=1.57079632679 effort=28 velocity=-1 -> lower=-1.57079632679 upper=1.57079632679 effort=28 velocity=24
